File: kicad/MCU.sch (KiCad schematic (older format))
At the start: 8 parts, among them J1 USB_B_Micro, U33 STM32F745VGHx, U36 S25FL064L, Y1 CSTNE8M00G550000R0

Commit message: modified:   kicad/MCU.sch 	modified:   kicad/OSD.sch 	modified:   kicad/Sensors.sch 	modified:   kicad/sym-lib-table 	modified:   kicad/ultimateFC-cache.lib 	modified:   kicad/ultimateFC.kicad_pcb 	modified:   kicad/ultimateFC.pro 	modified:   kicad/ultimateFC.sch 	modified:   simulations/video_amp.asc 	new file:   simulations/video_amp.log 	new file:   simulations/video_amp.op.raw 	new file:   simulations/video_amp.raw
Parts:
- removed D2: D_Schottky, Diode_SMD:D_0402_1005Metric, symbol Device:D_Schottky
- removed J1: USB_B_Micro, Connector_USB:USB_Micro-B_Molex_47346-0001, symbol Connector:USB_B_Micro
- removed R4, R5, R6: R, Resistor_SMD:R_0201_0603Metric, symbol Device:R
- removed U33: STM32F745VGHx, Package_BGA:TFBGA-100_8x8mm_Layout10x10_P0.8mm, symbol MCU_ST_STM32F7:STM32F745VGHx
- removed U36: S25FL064L, Package_SON:WSON-8_4x4mm_P0.8mm, symbol Memory_Flash:W25Q128JVS
- removed Y1: CSTNE8M00G550000R0, Crystal:Resonator_SMD_muRata_CSTxExxV-3Pin_3.0x1.1mm, symbol Device:Crystal_GND2
Connections:
- net labels removed: (TIM1_CH2), (TIM1_CH3), (TIM1_CH4), (UART5_RX), (UART5_TX), (UART7_RX), (UART7_TX), (UART8_RX), (UART8_TX), (USART6_RX), (USART6_TX), +3.3V, +5V, ADC1_10, ADC1_5, GND, I2C1_SCL, I2C1_SDA, I2C2_SCL, I2C2_SDA, I2C3_SCA, I2C3_SCL, SD_det, SPI1_MISO, SPI1_MOSI, SPI1_NSS, SPI1_SCK, SPI2_MISO, SPI2_MOSI, SPI2_NSS, SPI2_SCK, SPI3_MISO, SPI3_MOSI, SPI3_NSS, SPI3_SCK, TIM1_CH1, TIM4_CH1, TIM4_CH2, TIM4_CH3, TIM4_CH4, UART4_RX, UART4_TX, USART1_RX, USART1_TX, USART2_RX, USART2_TX, USART3_RX, USART3_TX
- wire segments 111 -> 0
- no-connect marks 2 -> 0
Other:
- note removed: "Internal Pullup on BOOT0:\n30k...50k"
- note removed: "Internal Pullup on NRST:\n30k...50k"
- note removed: "Pin assignments in parantheses (...) not checked in CubeMX!"
- note removed: "assign SPI instance"
- note removed: "clarify"
- note removed: "issue #1"
- note removed: "issue #2"
