File: kicad/Sensors.sch (KiCad schematic (older format))
At the start: 5 parts, among them U34 ICM-20602, U35 ZOE-M8Q_ZOE-M8Q, X1 Molex_734120110

Commit message: modified:   kicad/MCU.sch 	modified:   kicad/OSD.sch 	modified:   kicad/Sensors.sch 	modified:   kicad/sym-lib-table 	modified:   kicad/ultimateFC-cache.lib 	modified:   kicad/ultimateFC.kicad_pcb 	modified:   kicad/ultimateFC.pro 	modified:   kicad/ultimateFC.sch 	modified:   simulations/video_amp.asc 	new file:   simulations/video_amp.log 	new file:   simulations/video_amp.op.raw 	new file:   simulations/video_amp.raw
Parts:
- removed D1: True Green, LED_SMD:LED_0201_0603Metric, symbol Device:LED
- removed R3: 470R, Resistor_SMD:R_0201_0603Metric, symbol Device:R
- removed U34: ICM-20602, Package_LGA:LGA-16_3x3mm_P0.5mm_LayoutBorder3x5y, symbol Sensor_Motion:ICM-20602
- removed U35: ZOE-M8Q_ZOE-M8Q, ultimateFC:ZOE-M8, symbol lib_ultimateFC:ZOE-M8Q_ZOE-M8Q
- removed X1: Molex_734120110, ultimateFC:Molex_734120110, symbol lib_ultimateFC:Molex_734120110
Connections:
- net labels removed: +3.3V, GND
- wire segments 68 -> 0
- no-connect marks 24 -> 0
Other:
- note removed: "MISO"
- note removed: "MOSI"
- note removed: "SCK"
- note removed: "assign IMU INT line"
- note removed: "assign SPI instance"
- note removed: "assign UART instance"
- note removed: "connect to castellated pad"
