File: kicad/ultimateFC_v2.kicad_pcb (KiCad board)
At the start: 8 copper layers, 30.4 x 25.2 mm, 192 parts, among them J1 USB_B_Micro, J2 10132797-011100LF, J3 10132797-011100LF, J4 10132797-011100LF, J5 10132797-011100LF, J6 10132797-011100LF, Q1 DMP2066LSN-7, U1 EFM8BB21F16G-C-QFN20R, U10 NCP81253MNTBG, U11 SiZ200DT, U12 NCP81253MNTBG, U13 SiZ200DT, U14 TPS62821, U15 SiZ200DT, U16 NCP81253MNTBG, U17 NCP81253MNTBG, U18 NCP81253MNTBG, U19 NCP81253MNTBG, U2 EFM8BB21F16G-C-QFN20R, U20 SiZ200DT, U21 SiZ200DT, U22 SiZ200DT, U23 SiZ200DT, U24 EFM8BB21F16G-C-QFN20R, U25 NCP81253MNTBG, U26 SiZ200DT, U27 NCP81253MNTBG, U28 NCP81253MNTBG, U29 SiZ200DT, U3 NCP81253MNTBG, U30 SiZ200DT, U31 INA186, U32 LMR33630CQRNX, U33 STM32F745VGHx, U34 AB7456, U35 ZOE-M8Q_ZOE-M8Q, U36 ICM-20602, U37 S25FL064L, U39 BMP280, U4 SiZ200DT, U6 EFM8BB21F16G-C-QFN20R, U7 NCP81253MNTBG, U8 SiZ200DT, U9 NCP81253MNTBG, X1 Molex_734120110, Y1 CSTNE8M00G550000R0, Y2 ECS-270-8-47Q-CES-TR

Commit message: updated to version 2
Parts:
- removed the REF** at (197.1, 64.1) (x2)
- added REF**: Fiducial_0.5mm_Dia_1mm_Outer, Fiducial:Fiducial_0.5mm_Dia_1mm_Outer, F.Cu at (197.1, 64.1)
- added REF**: Fiducial_0.5mm_Dia_1mm_Outer, Fiducial:Fiducial_0.5mm_Dia_1mm_Outer, B.Cu at (197.1, 64.1)
Changed lines of the file:
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@@
   )
   (setup
-    (last_trace_width 0.1)
+    (last_trace_width 0.25)
     (user_trace_width 0.1)
     (user_trace_width 0.2)
@@
     (arrow2b (pts (xy 166 62) (xy 166.586421 63.126504)))
   )
+  (via (at 169.875 81.2) (size 0.4) (drill 0.2) (layers F.Cu B.Cu) (net 271))
+  (via (at 195.95 74.65) (size 0.4) (drill 0.2) (layers F.Cu B.Cu) (net 8))
+  (via (at 196.3 74.9) (size 0.4) (drill 0.2) (layers F.Cu B.Cu) (net 8))
+  (via (at 195.45 82.675) (size 0.4) (drill 0.2) (layers F.Cu B.Cu) (net 4))
   (via (at 195.45 80.625) (size 0.4) (drill 0.2) (layers F.Cu B.Cu) (net 1))
   (via (at 196.675 61.325) (size 0.4) (drill 0.2) (layers F.Cu B.Cu) (net 1))
+  (via (at 195.05 82) (size 0.4) (drill 0.2) (layers F.Cu B.Cu) (net 4))
+  (via (at 196.275 81.3) (size 0.4) (drill 0.2) (layers F.Cu B.Cu) (net 4))
+  (via (at 195.775 82) (size 0.4) (drill 0.2) (layers F.Cu B.Cu) (net 4))
+  (via (at 197 81.299999) (size 0.4) (drill 0.2) (layers F.Cu B.Cu) (net 4))
   (via (at 195.05 81.3) (size 0.4) (drill 0.2) (layers F.Cu B.Cu) (net 1))
   (via (at 195.775 81.3) (size 0.4) (drill 0.2) (layers F.Cu B.Cu) (net 1))
@@
   (via (at 195.775 62.7) (size 0.4) (drill 0.2) (layers F.Cu B.Cu) (net 1))
   (via (at 196.275 62) (size 0.4) (drill 0.2) (layers F.Cu B.Cu) (net 1))
+  (via (at 196.275 62.7) (size 0.4) (drill 0.2) (layers F.Cu B.Cu) (net 4))
   (via (at 170.35 77.450001) (size 0.4) (drill 0.2) (layers F.Cu B.Cu) (net 1))
   (via (at 170.85 76.95) (size 0.4) (drill 0.2) (layers F.Cu B.Cu) (net 1))
@@
   (segment (start 169.1625 65.7) (end 169.937045 64.925455) (width 0.1) (layer B.Cu) (net 1))
   (segment (start 169.937045 64.925455) (end 169.937045 64.882739) (width 0.1) (layer B.Cu) (net 1))
+  (via (at 196.625 63.375) (size 0.4) (drill 0.2) (layers F.Cu B.Cu) (net 4))
   (via (at 172.55 77.450001) (size 0.4) (drill 0.2) (layers F.Cu B.Cu) (net 2))
   (via (at 173.05 76.95) (size 0.4) (drill 0.2) (layers F.Cu B.Cu) (net 2))
@@
   (segment (start 195.5 75.8) (end 195.5 76.155263) (width 0.1) (layer B.Cu) (net 2))
   (via (at 196.100148 76.472569) (size 0.4) (drill 0.2) (layers F.Cu B.Cu) (net 2))
+  (segment (start 169.65 67.45) (end 169.65 67.4) (width 0.1) (layer F.Cu) (net 277))
   (segment (start 188.39 78.1) (end 188.470339 78.1) (width 0.1) (layer B.Cu) (net 2))
   (segment (start 187.86 78.63) (end 188.39 78.1) (width 0.1) (layer B.Cu) (net 2))
@@
   (segment (start 180.392519 76.362519) (end 179.730371 76.362519) (width 0.1) (layer B.Cu) (net 3))
   (via (at 171.01 72.91) (size 0.4) (drill 0.2) (layers F.Cu B.Cu) (net 3))
-  (via (at 195.45 82.675) (size 0.4) (drill 0.2) (layers F.Cu B.Cu) (net 4))
-  (via (at 195.05 82) (size 0.4) (drill 0.2) (layers F.Cu B.Cu) (net 4))
-  (via (at 196.275 81.3) (size 0.4) (drill 0.2) (layers F.Cu B.Cu) (net 4))
-  (via (at 195.775 82) (size 0.4) (drill 0.2) (layers F.Cu B.Cu) (net 4))
-  (via (at 197 81.299999) (size 0.4) (drill 0.2) (layers F.Cu B.Cu) (net 4))
-  (via (at 196.275 62.7) (size 0.4) (drill 0.2) (layers F.Cu B.Cu) (net 4))
-  (via (at 196.625 63.375) (size 0.4) (drill 0.2) (layers F.Cu B.Cu) (net 4))
   (segment (start 183.972436 81.932556) (end 183.972436 81.939725) (width 0.1) (layer F.Cu) (net 4))
   (segment (start 183.98 81.924992) (end 183.972436 81.932556) (width 0.1) (layer F.Cu) (net 4))
@@
   (segment (start 189.126688 70.549999) (end 187.699999 70.549999) (width 0.1) (layer B.Cu) (net 7))
   (segment (start 187.699999 70.549999) (end 187.449999 70.299999) (width 0.1) (layer B.Cu) (net 7))
-  (via (at 195.95 74.65) (size 0.4) (drill 0.2) (layers F.Cu B.Cu) (net 8))
-  (via (at 196.3 74.9) (size 0.4) (drill 0.2) (layers F.Cu B.Cu) (net 8))
   (via (at 197.1 75.4) (size 0.4) (drill 0.2) (layers F.Cu B.Cu) (net 8))
   (via (at 196.7 75.4) (size 0.4) (drill 0.2) (layers F.Cu B.Cu) (net 8))
@@
   (segment (start 188.33 75.98) (end 188.05 75.7) (width 0.1) (layer B.Cu) (net 137))
   (segment (start 188.33 76.37) (end 188.33 75.98) (width 0.1) (layer B.Cu) (net 137))
+  (segment (start 181.77 78.2) (end 181.77 78.123542) (width 0.1) (layer B.Cu) (net 281))
+  (segment (start 181.77 78.123542) (end 181.761182 78.114724) (width 0.1) (layer B.Cu) (net 281))
   (segment (start 179.61571 79.15429) (end 179.42 79.35) (width 0.1) (layer F.Cu) (net 139))
   (segment (start 179.79499 78.97501) (end 179.61571 79.15429) (width 0.1) (layer F.Cu) (net 139))
@@
   (segment (start 168.919999 79.779999) (end 168.919999 79.639999) (width 0.1) (layer In6.Cu) (net 270))
   (segment (start 168.919999 79.639999) (end 168.86 79.58) (width 0.1) (layer In6.Cu) (net 270))
-  (via (at 169.875 81.2) (size 0.4) (drill 0.2) (layers F.Cu B.Cu) (net 271))
   (segment (start 173.495648 74.404352) (end 173.495648 74.407261) (width 0.1) (layer F.Cu) (net 271))
   (segment (start 173.6 74.3) (end 173.495648 74.404352) (width 0.1) (layer F.Cu) (net 271))
@@
   (segment (start 171.344999 75.454999) (end 171.79 75.9) (width 0.25) (layer B.Cu) (net 276))
   (segment (start 171.344999 75.350001) (end 171.344999 75.454999) (width 0.25) (layer B.Cu) (net 276))
-  (segment (start 169.65 67.45) (end 169.65 67.4) (width 0.1) (layer F.Cu) (net 277))
   (via (at 179.39 68.57) (size 0.4) (drill 0.2) (layers F.Cu B.Cu) (net 277))
   (segment (start 179.575 70) (end 179.575 68.755) (width 0.1) (layer F.Cu) (net 277))
@@
   (segment (start 188.327541 67.149859) (end 187.9774 67.5) (width 0.1) (layer In6.Cu) (net 280))
   (segment (start 187.9774 67.5) (end 185.118002 67.5) (width 0.1) (layer In6.Cu) (net 280))
-  (segment (start 181.77 78.2) (end 181.77 78.123542) (width 0.1) (layer B.Cu) (net 281))
-  (segment (start 181.77 78.123542) (end 181.761182 78.114724) (width 0.1) (layer B.Cu) (net 281))
   (via (at 188.293994 76.864018) (size 0.4) (drill 0.2) (layers F.Cu B.Cu) (net 281))
   (segment (start 188.33 76.97) (end 188.33 76.900024) (width 0.1) (layer B.Cu) (net 281))
