File: kicad/ultimateFC.sch (KiCad schematic (older format))
At the start: 142 parts, among them J2 10132797-011100LF, J3 10132797-011100LF, J4 10132797-011100LF, J5 10132797-011100LF, J6 Conn_02x10_Counter_Clockwise, U1 EFM8BB21F16G-C-QFN20R, U10 NCP81253MNTBG, U11 SIZ322DT-T1-GE3, U12 NCP81253MNTBG, U13 SIZ322DT-T1-GE3, U14 TPS62821, U15 SIZ322DT-T1-GE3, U16 NCP81253MNTBG, U17 NCP81253MNTBG, U18 NCP81253MNTBG, U19 NCP81253MNTBG, U2 EFM8BB21F16G-C-QFN20R, U20 SIZ322DT-T1-GE3, U21 SIZ322DT-T1-GE3, U22 SIZ322DT-T1-GE3, U23 SIZ322DT-T1-GE3, U24 EFM8BB21F16G-C-QFN20R, U25 NCP81253MNTBG, U26 SIZ322DT-T1-GE3, U27 NCP81253MNTBG, U28 NCP81253MNTBG, U29 SIZ322DT-T1-GE3, U3 NCP81253MNTBG, U30 SIZ322DT-T1-GE3, U31 INA186, U32 LMR33630CQRNX, U4 SIZ322DT-T1-GE3, U5 TPS630701, U6 EFM8BB21F16G-C-QFN20R, U7 NCP81253MNTBG, U8 SIZ322DT-T1-GE3, U9 NCP81253MNTBG

Commit message: modified:   kicad/MCU.sch 	modified:   kicad/OSD.sch 	modified:   kicad/Sensors.sch 	modified:   kicad/sym-lib-table 	modified:   kicad/ultimateFC-cache.lib 	modified:   kicad/ultimateFC.kicad_pcb 	modified:   kicad/ultimateFC.pro 	modified:   kicad/ultimateFC.sch 	modified:   simulations/video_amp.asc 	new file:   simulations/video_amp.log 	new file:   simulations/video_amp.op.raw 	new file:   simulations/video_amp.raw
Parts:
- removed J6: Conn_02x10_Counter_Clockwise, ultimateFC:10132797-021100LF, symbol Connector_Generic:Conn_02x10_Counter_Clockwise
- added C47: 100nF, Capacitor_SMD:C_0201_0603Metric, symbol Device:C_Small
- added C48: 47µF, Capacitor_SMD:C_0603_1608Metric, symbol Device:CP_Small
- added C49: 22µF, Capacitor_SMD:C_0603_1608Metric, symbol Device:CP_Small
- added C50, C51, C52, C53: 2.2µF, Capacitor_SMD:C_0402_1005Metric, symbol Device:C
- added D1: True Green, LED_SMD:LED_0201_0603Metric, symbol Device:LED
- added D2: D_Schottky, Diode_SMD:D_0402_1005Metric, symbol Device:D_Schottky
- added D3: Blue, LED_SMD:LED_0201_0603Metric, symbol Device:LED
- added D4: Red, LED_SMD:LED_0201_0603Metric, symbol Device:LED
- added J1: USB_B_Micro, Connector_USB:USB_Micro-B_Molex_47346-0001, symbol Connector:USB_B_Micro
- added J6: 10132797-011100LF, ultimateFC:10132797-011100LF, symbol Connector_Generic:Conn_02x05_Counter_Clockwise
- added R10, R5: 470R, Resistor_SMD:R_0201_0603Metric, symbol Device:R
- added R3, R6: 75R, Resistor_SMD:R_0402_1005Metric, symbol Device:R
- added R4, R7, R8: R, Resistor_SMD:R_0201_0603Metric, symbol Device:R
- added R9: 100R, Resistor_SMD:R_0201_0603Metric, symbol Device:R
- added TP23, TP24, TP25, TP26, TP27, TP28, TP29, TP30: pad, TestPoint:TestPoint_Pad_1.0x1.0mm, symbol Connector:TestPoint_Alt
- added U33: STM32F745VGHx, Package_BGA:TFBGA-100_8x8mm_Layout10x10_P0.8mm, symbol MCU_ST_STM32F7:STM32F745VGHx
- added U34: AB7456, Package_SO:TSSOP-28_4.4x9.7mm_P0.65mm, symbol lib_ultimateFC:AB7456
- added U35: ZOE-M8Q_ZOE-M8Q, ultimateFC:ZOE-M8, symbol lib_ultimateFC:ZOE-M8Q_ZOE-M8Q
- added U36: ICM-20602, Package_LGA:LGA-16_3x3mm_P0.5mm_LayoutBorder3x5y, symbol Sensor_Motion:ICM-20602
- added U37: S25FL064L, Package_SON:WSON-8_4x4mm_P0.8mm, symbol Memory_Flash:W25Q128JVS
- added U38: LIS3MDL, Package_LGA:LGA-12_2x2mm_P0.5mm, symbol own_devices:LIS3MDL
- added U39: BMP280, Package_LGA:Bosch_LGA-8_2x2.5mm_P0.65mm_ClockwisePinNumbering, symbol Sensor_Pressure:BMP280
- added X1: Molex_734120110, ultimateFC:Molex_734120110, symbol lib_ultimateFC:Molex_734120110
- added Y1: CSTNE8M00G550000R0, Crystal:Resonator_SMD_muRata_CSTxExxV-3Pin_3.0x1.1mm, symbol Device:Crystal_GND2
- added Y2: 27M, Crystal:Crystal_SMD_MicroCrystal_CM9V-T1A-2Pin_1.6x1.0mm, symbol Device:Crystal_Small
- R47: footprint Resistor_SMD:R_0201_0603Metric -> Resistor_SMD:R_0402_1005Metric
- U11, U13, U15, U20, U21, U22, U23, U26, U29, U30, U4, U8: value SIZ322DT-T1-GE3 -> SiZ200DT
Connections:
- net labels added: (TIM1_CH3), (TIM1_CH4), (UART5_RX), (UART7_RX), (UART7_TX), (UART8_RX), (UART8_TX), (USART6_RX), (USART6_TX), ADC1_10, ADC1_5, CS_BERGSTAK20, CS_FLASH, CS_GYRO, CS_OSD, I2C2_SCL, I2C2_SDA, INT_GYRO, MISO_FLASH, MISO_GYRO, MISO_OSD, MOSI_FLASH, MOSI_GYRO, MOSI_OSD, MOTOR1, MOTOR2, MOTOR3, MOTOR4, MP_PIN5, MP_PIN6, OSD_VIDEO_IN, OSD_VIDEO_OUT, SCLK_FLASH, SCLK_GYRO, SCLK_OSD, SD_det, SPI1_NSS, SPI2_MISO, SPI2_MOSI, SPI2_NSS, SPI2_SCK, SPI3_MISO, SPI3_MOSI, SPI3_NSS, SPI3_SCK, SPI4_MISO, SPI4_MOSI, SPI4_NSS, SPI4_SCK, TIM4_CH1, TIM4_CH2, TIM4_CH3, TIM4_CH4, UART7_RX, UART7_TX, UART8_RX, UART8_TX, UC_LED_1, UC_LED_2, USART1_RX, USART1_TX, USART2_TX, USART3_RX, USART3_TX
- net labels removed: ESC5, ESC6, SPI1_CS, SPI1_MISO, SPI1_MOSI, SPI_1SCK, UART2_RX, UART2_TX, USB_N, USB_P, Video_in, Video_out
- wire segments 621 -> 857
- no-connect marks 16 -> 43
Other:
- note added: "Changed to 22u (see video_amp.asc simulation file)"
- note added: "Flash"
- note added: "Gyro"
- note added: "Interface"
- note added: "Internal Pullup on BOOT0:\n30k...50k"
- note added: "Internal Pullup on NRST:\n30k...50k"
- note added: "MISO"
- note added: "MOSI"
- note added: "Not used (was Bergstak 20)"
- note added: "OSD"
- note added: "Pin assignments in parantheses (...) not checked in CubeMX!"
- note added: "Ressource\n"
- note added: "SCK"
- note added: "SPI 1"
- note added: "SPI 2"
- note added: "SPI 3"
- note added: "SPI 4"
- note added: "The Capacitance change due to DC bias has to be considered \n(up to 4V on C47 und up to 2 V over C48 according to the simulation)\nTherefore chnage to Tantals"
- note added: "UART4\n"
- note added: "UART5\n"
- note added: "UART7\n"
- note added: "UART8\n"
- note added: "USART1\n"
- note added: "USART2\n"
- note added: "USART3\n\n"
- note added: "USART6\n"
- note added: "assign IMU INT line"
- note added: "assign SPI instance"
- note added: "clarify"
- note added: "connect to castellated pad"
- note added: "issue #1"
- note added: "issue #2"
- moved on the sheet: C1, C10, C11, C12, C13, C14, C15, C16, C17, C18, C19, C2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

Commit message: status 2021-03-10
Parts:
- added C54: 100nF, Capacitor_SMD:C_0201_0603Metric, symbol Device:C
- added L4: 39nH, Inductor_SMD:L_0201_0603Metric, symbol Device:L
- added R11: 10R, Resistor_SMD:R_0201_0603Metric, symbol Device:R
- C24, C25, C45, C46: value 10µF -> 100nF; footprint Capacitor_SMD:C_0603_1608Metric -> ultimateFC:C_AVX_Super_Low_ESL; Mfr.No: (none) -> W2L16D105MAT1A
Connections:
- net labels added: NO_ADC_PIN
- net labels removed: ADC1_10
- wire segments 857 -> 862
Other:
- note added: "Add 2k7 pulldown"
- note added: "FLash hinzufügen?"
- note added: "NEW"
- note added: "Pullups für I2C"
- note added: "Specify Quartz"
- note added: "Wechsel auf TFM252012ALMA1R0MTAA wär nicht verkehrt"
- note removed: "Internal Pullup on BOOT0:\n30k...50k"
- moved on the sheet: X1
Changed lines of the file:
@@
 $EndComp
 $Comp
-L Device:C C25
-U 1 1 5E77E8A2
-P 9250 12325
-F 0 "C25" H 9365 12371 50  0000 L CNN
-F 1 "10µF" H 9365 12280 50  0000 L CNN
-F 2 "Capacitor_SMD:C_0603_1608Metric" H 9288 12175 50  0001 C CNN
-F 3 "~" H 9250 12325 50  0001 C CNN
-F 4 "25V" H 9250 12325 50  0001 C CNN "Spannung"
-F 5 "X5R" H 9250 12325 50  0001 C CNN "Dielektrikum"
-	1    9250 12325
-	1    0    0    -1
-$EndComp
-$Comp
 L power:GND #PWR0238
 U 1 1 5E77F592
@@
 $EndComp
 $Comp
-L Device:C C24
-U 1 1 5E77DDF4
-P 9250 11550
-F 0 "C24" H 9365 11596 50  0000 L CNN
-F 1 "10µF" H 9365 11505 50  0000 L CNN
-F 2 "Capacitor_SMD:C_0603_1608Metric" H 9288 11400 50  0001 C CNN
-F 3 "~" H 9250 11550 50  0001 C CNN
-F 4 "25V" H 9250 11550 50  0001 C CNN "Spannung"
-F 5 "X5R" H 9250 11550 50  0001 C CNN "Dielektrikum"
-	1    9250 11550
-	1    0    0    -1
-$EndComp
-$Comp
 L Device:C C22
 U 1 1 5E77CD3C
@@
 $EndComp
 $Comp
-L Device:C C46
-U 1 1 5F3EBE44
-P 9650 12325
-F 0 "C46" H 9765 12371 50  0000 L CNN
-F 1 "10µF" H 9765 12280 50  0000 L CNN
-F 2 "Capacitor_SMD:C_0603_1608Metric" H 9688 12175 50  0001 C CNN
-F 3 "~" H 9650 12325 50  0001 C CNN
-F 4 "25V" H 9650 12325 50  0001 C CNN "Spannung"
-F 5 "X5R" H 9650 12325 50  0001 C CNN "Dielektrikum"
-	1    9650 12325
-	1    0    0    -1
-$EndComp
-$Comp
 L power:GND #PWR0292
 U 1 1 5F3EBE4A
@@
 	1    0    0    -1
 $EndComp
-$Comp
-L Device:C C45
-U 1 1 5F3EBE64
-P 9650 11550
-F 0 "C45" H 9765 11596 50  0000 L CNN
-F 1 "10µF" H 9765 11505 50  0000 L CNN
-F 2 "Capacitor_SMD:C_0603_1608Metric" H 9688 11400 50  0001 C CNN
-F 3 "~" H 9650 11550 50  0001 C CNN
-F 4 "25V" H 9650 11550 50  0001 C CNN "Spannung"
-F 5 "X5R" H 9650 11550 50  0001 C CNN "Dielektrikum"
-	1    9650 11550
-	1    0    0    -1
-$EndComp
 $Sheet
 S 31925 250  2550 3050
@@
 L lib_ultimateFC:Molex_734120110 X?
 U 1 1 5F4E0E52
-P 24725 10825
+P 25375 11125
 AR Path="/5ED2E134/5F4E0E52" Ref="X?"  Part="1"
 AR Path="/5F4E0E52" Ref="X1"  Part="1"
-F 0 "X1" H 24594 10865 50  0000 R CNN
-F 1 "Molex_734120110" H 24594 10774 50  0000 R CNN
-F 2 "ultimateFC:Molex_734120110" H 24725 10825 50  0001 L BNN
-F 3 "734120110" H 24725 10825 50  0001 L BNN
-F 4 "https://www.digikey.com/product-detail/en/molex/0734120110/WM5587CT-ND/1894612?utm_source=snapeda&utm_medium=aggregator&utm_campaign=symbol" H 24725 10825 50  0001 L BNN "Field4"
-F 5 "None" H 24725 10825 50  0001 L BNN "Field5"
-F 6 "Molex" H 24725 10825 50  0001 L BNN "Field6"
-F 7 "WM5587CT-ND" H 24725 10825 50  0001 L BNN "Field7"
-F 8 "Conn Micro Coaxial RCP 0Hz to 6GHz 50Ohm Solder ST SMD Gold T/R" H 24725 10825 50  0001 L BNN "Field8"
-	1    24725 10825
+F 0 "X1" H 25244 11165 50  0000 R CNN
+F 1 "Molex_734120110" H 25244 11074 50  0000 R CNN
+F 2 "ultimateFC:Molex_734120110" H 25375 11125 50  0001 L BNN
+F 3 "734120110" H 25375 11125 50  0001 L BNN
+F 4 "https://www.digikey.com/product-detail/en/molex/0734120110/WM5587CT-ND/1894612?utm_source=snapeda&utm_medium=aggregator&utm_campaign=symbol" H 25375 11125 50  0001 L BNN "Field4"
+F 5 "None" H 25375 11125 50  0001 L BNN "Field5"
+F 6 "Molex" H 25375 11125 50  0001 L BNN "Field6"
+F 7 "WM5587CT-ND" H 25375 11125 50  0001 L BNN "Field7"
+F 8 "Conn Micro Coaxial RCP 0Hz to 6GHz 50Ohm Solder ST SMD Gold T/R" H 25375 11125 50  0001 L BNN "Field8"
+	1    25375 11125
 	-1   0    0    -1
 $EndComp
@@
 	24525 14225 24425 14225
 Wire Wire Line
-	24425 11125 24625 10825
+	24425 11125 24800 11125
 $Comp
 L power:GND #PWR?
 U 1 1 5F4E0E7C
-P 24625 11300
+P 25275 11600
 AR Path="/5ED2E134/5F4E0E7C" Ref="#PWR?"  Part="1"
 AR Path="/5F4E0E7C" Ref="#PWR0296"  Part="1"
-F 0 "#PWR0296" H 24625 11050 50  0001 C CNN
-F 1 "GND" H 24630 11127 50  0000 C CNN
-F 2 "" H 24625 11300 50  0001 C CNN
-F 3 "" H 24625 11300 50  0001 C CNN
-	1    24625 11300
+F 0 "#PWR0296" H 25275 11350 50  0001 C CNN
+F 1 "GND" H 25280 11427 50  0000 C CNN
+F 2 "" H 25275 11600 50  0001 C CNN
+F 3 "" H 25275 11600 50  0001 C CNN
+	1    25275 11600
 	1    0    0    -1
 $EndComp
@@
 Wire Wire Line
 	21825 1825 20625 1825
-Text Notes 19975 1875 0    50   ~ 0
-Internal Pullup on BOOT0:\n30k...50k
 $Comp
 L power:GND #PWR?
@@
 Wire Wire Line
 	23725 2425 24375 2425
-Text Label 23825 2425 0    50   ~ 0
-ADC1_10
+Text Label 23825 2425 0    50   ~ 10
+NO_ADC_PIN
 Wire Wire Line
 	23725 1825 24375 1825
@@
 Wire Notes Line
 	28925 4800 28925 6925
-Text GLabel 24375 1825 2    50   Input ~ 0
-CS_BERGSTAK20
 Text GLabel 25325 8425 0    50   Input ~ 0
 CS_FLASH
@@
 	27350 11925 27350 11825
 Wire Wire Line
-	24625 10925 24625 11300
+	25275 11225 25275 11600
 $Comp
 L Connector:TestPoint_Alt TP25
@@
 Text GLabel 24375 1925 2    50   Input ~ 0
 curr_sig
-Text GLabel 24375 2425 2    50   Input ~ 0
-vol_sig
 Text GLabel 2375 8225 0    50   Input ~ 0
 MOTOR2
@@
 	-1   0    0    1
 $EndComp
+$Comp
+L Device:C C45
+U 1 1 600A0CAC
+P 9650 11550
+F 0 "C45" H 9765 11596 50  0000 L CNN
+F 1 "100nF" H 9765 11505 50  0000 L CNN
+F 2 "ultimateFC:C_AVX_Super_Low_ESL" H 9688 11400 50  0001 C CNN
+F 3 "~" H 9650 11550 50  0001 C CNN
+F 4 "25V" H 9650 11550 50  0001 C CNN "Spannung"
+F 5 "X5R" H 9650 11550 50  0001 C CNN "Dielektrikum"
+F 6 "W2L16D105MAT1A" H 9650 11550 50  0001 C CNN "Mfr.No:"
+	1    9650 11550
+	-1   0    0    -1
+$EndComp
+$Comp
+L Device:C C24
+U 1 1 600A3B07
+P 9250 11550
+F 0 "C24" H 9365 11596 50  0000 L CNN
+F 1 "100nF" H 9365 11505 50  0000 L CNN
+F 2 "ultimateFC:C_AVX_Super_Low_ESL" H 9288 11400 50  0001 C CNN
+F 3 "~" H 9250 11550 50  0001 C CNN
+F 4 "25V" H 9250 11550 50  0001 C CNN "Spannung"
+F 5 "X5R" H 9250 11550 50  0001 C CNN "Dielektrikum"
+F 6 "W2L16D105MAT1A" H 9250 11550 50  0001 C CNN "Mfr.No:"
+	1    9250 11550
+	1    0    0    1
+$EndComp
+$Comp
+L Device:C C25
+U 1 1 600A3F04
+P 9250 12325
+F 0 "C25" H 9365 12371 50  0000 L CNN
+F 1 "100nF" H 9365 12280 50  0000 L CNN
+F 2 "ultimateFC:C_AVX_Super_Low_ESL" H 9288 12175 50  0001 C CNN
+F 3 "~" H 9250 12325 50  0001 C CNN
+F 4 "25V" H 9250 12325 50  0001 C CNN "Spannung"
+F 5 "X5R" H 9250 12325 50  0001 C CNN "Dielektrikum"
+F 6 "W2L16D105MAT1A" H 9250 12325 50  0001 C CNN "Mfr.No:"
+	1    9250 12325
+	1    0    0    1
+$EndComp
+$Comp
+L Device:C C46
+U 1 1 600A43DB
+P 9650 12325
+F 0 "C46" H 9765 12371 50  0000 L CNN
+F 1 "100nF" H 9765 12280 50  0000 L CNN
+F 2 "ultimateFC:C_AVX_Super_Low_ESL" H 9688 12175 50  0001 C CNN
+F 3 "~" H 9650 12325 50  0001 C CNN
+F 4 "25V" H 9650 12325 50  0001 C CNN "Spannung"
+F 5 "X5R" H 9650 12325 50  0001 C CNN "Dielektrikum"
+F 6 "W2L16D105MAT1A" H 9650 12325 50  0001 C CNN "Mfr.No:"
+	1    9650 12325
+	-1   0    0    -1
+$EndComp
+$Comp
+L Device:C C54
+U 1 1 600A769D
+P 25150 10500
+F 0 "C54" H 25265 10546 50  0000 L CNN
+F 1 "100nF" H 25265 10455 50  0000 L CNN
+F 2 "Capacitor_SMD:C_0201_0603Metric" H 25188 10350 50  0001 C CNN
+F 3 "~" H 25150 10500 50  0001 C CNN
+F 4 "X5R" H 25150 10500 50  0001 C CNN "Dielektrikum"
+F 5 "16V" H 25150 10500 50  0001 C CNN "Spannung"
+	1    25150 10500
+	1    0    0    -1
+$EndComp
+$Comp
+L Device:R R11
+U 1 1 600A8828
+P 25150 10200
+F 0 "R11" V 25050 10175 50  0000 L CNN
+F 1 "10R" V 25150 10150 50  0000 L CNN
+F 2 "Resistor_SMD:R_0201_0603Metric" V 25080 10200 50  0001 C CNN
+F 3 "~" H 25150 10200 50  0001 C CNN
+	1    25150 10200
+	-1   0    0    1
+$EndComp
+$Comp
+L power:GND #PWR0330
+U 1 1 600A9EF7
+P 25150 10650
+F 0 "#PWR0330" H 25150 10400 50  0001 C CNN
+F 1 "GND" H 25155 10477 50  0000 C CNN
+F 2 "" H 25150 10650 50  0001 C CNN
+F 3 "" H 25150 10650 50  0001 C CNN
+	1    25150 10650
+	1    0    0    -1
+$EndComp
+$Comp
+L power:+3.3V #PWR0331
+U 1 1 600AAD39
+P 25150 10050
+F 0 "#PWR0331" H 25150 9900 50  0001 C CNN
+F 1 "+3.3V" H 25165 10223 50  0000 C CNN
+F 2 "" H 25150 10050 50  0001 C CNN
+F 3 "" H 25150 10050 50  0001 C CNN
+	1    25150 10050
+	1    0    0    -1
+$EndComp
+$Comp
+L Device:L L4
+U 1 1 600AB5C6
+P 24800 10700
+F 0 "L4" H 24853 10746 50  0000 L CNN
+F 1 "39nH" H 24853 10655 50  0000 L CNN
+F 2 "Inductor_SMD:L_0201_0603Metric" H 24800 10700 50  0001 C CNN
+F 3 "~" H 24800 10700 50  0001 C CNN
+	1    24800 10700
+	1    0    0    -1
+$EndComp
+Wire Wire Line
+	24800 10850 24800 11125
+Connection ~ 24800 11125
+Wire Wire Line
+	24800 11125 25275 11125
+Wire Wire Line
+	25150 10350 24800 10350
+Wire Wire Line
+	24800 10350 24800 10550
+Connection ~ 25150 10350
+Text Notes 3800 13825 0    50   ~ 0
+Wechsel auf TFM252012ALMA1R0MTAA wär nicht verkehrt
+Wire Notes Line
+	4400 14000 4400 13900
+Wire Notes Line
+	4400 13900 4375 13900
+Text Notes 25800 12625 0    50   ~ 10
+Specify Quartz
+Text Notes 20100 2075 0    50   ~ 10
+Add 2k7 pulldown
+Text Notes 22275 12125 0    50   ~ 10
+FLash hinzufügen?
+Text Notes 29125 7675 0    50   ~ 10
+Pullups für I2C
+Text GLabel 24375 5325 2    50   Input ~ 0
+vol_sig
+Text GLabel 24375 1825 2    50   Input ~ 0
+CS_BERGSTAK20
+Wire Wire Line
+	23725 5325 24375 5325
+Text Notes 24000 5325 0    50   ~ 10
+NEW
 $EndSCHEMATC

Commit message: updated to version 2
Parts:
- removed RN10, RN11, RN12, RN19: 1k, ultimateFC:EXB14V_0201x2, symbol Device:R_Pack02
- removed RN17, RN3, RN4, RN8: 2k, ultimateFC:EXB14V_0201x2, symbol Device:R_Pack02
- removed TP23, TP24, TP25, TP26, TP27, TP28: pad, TestPoint:TestPoint_Pad_1.0x1.0mm, symbol Connector:TestPoint_Alt
- added C55, C56: 2.2µF, Capacitor_SMD:C_0603_1608Metric, symbol Device:C
- added Q1: DMP2066LSN-7, Package_TO_SOT_SMD:SOT-323_SC-70, symbol Device:Q_PMOS_GSD
- added R12, R13, R14, R15, R16, R17, R18, R19, R20, R23, R24, R25, R26, R27, R28, R29, R30, R36, R37: 2k2, ultimateFC:R_0201_0603Metric_mod, symbol Device:R
- added R31, R32, R33, R34: 1k, ultimateFC:R_0201_0603Metric_mod, symbol Device:R
- added TP23: bridge, ultimateFC:solderbridge_tiny, symbol Device:Jumper
- C1, C2, C35, C36: price@100[€] (none) -> 0,077; price@10[€] (none) -> 0,114; price@1k[€] (none) -> 0,69
- C10, C16, C17, C18, C19, C29, C30, C31, C32, C34, C7, C9: Mfr.No: (none) -> GMK105BJ104KV-F; Spannung 16V -> 35V; price@100[€] (none) -> 0,019; price@10[€] (none) -> 0,077; price@1k[€] (none) -> 0,014
- C11, C39, C4, C8: Mfr.No: (none) -> AMK107ABJ106KAHT; Spannung 10V -> 6,3V; price@100[€] (none) -> 0,053; price@10[€] (none) -> 0,149; price@1k[€] (none) -> 0,041
- C12, C13: price@100[€] (none) -> 0,817; price@10[€] (none) -> 1,08; price@1k[€] (none) -> 0,544
- C14, C20, C41, C43: Dielektrikum X5R -> X7S; Mfr.No: W2L16D105MAT1A -> LLA215C70G105MA14K; price@100[€] (none) -> 0,149; price@10[€] (none) -> 0,248; price@1k[€] (none) -> 0,066
- C15, C21, C42, C44: value 1µF -> 2.2µF; Dielektrikum X5R -> X7S; Mfr.No: W2L16D105MAT1A -> LLA219C70G225MA01L; Spannung 6,3V -> 4V; price@100[€] (none) -> 0,127; price@10[€] (none) -> 0,213; price@1k[€] (none) -> 0,066
- C22, C23: value 10µF -> 2.2µF; Mfr.No: (none) -> GRM188R6YA475KE15D; Spannung 25V -> 35V; price@100[€] (none) -> 0,11; price@10[€] (none) -> 0,113; price@1k[€] (none) -> 0,104
- C24, C25, C45, C46: value 100nF -> 2.2µF; footprint ultimateFC:C_AVX_Super_Low_ESL -> Capacitor_SMD:C_0603_1608Metric; Mfr.No: W2L16D105MAT1A -> GRM188R6YA475KE15D; Spannung 25V -> 35V; price@100[€] (none) -> 0,11; price@10[€] (none) -> 0,113; price@1k[€] (none) -> 0,104
- C26, C27: price@100[€] (none) -> 0,351; price@10[€] (none) -> 0,512; price@1k[€] (none) -> 0,212
- C28, C3, C33, C38, C54: Mfr.No: (none) -> C0603X5R1E104K030BB; Spannung 16V -> 25V; price@100[€] (none) -> 0,037; price@10[€] (none) -> 0,03; price@1k[€] (none) -> 0,022
- C37: Mfr.No: (none) -> EMK105BJ105MVHF; price@100[€] (none) -> 0,025; price@10[€] (none) -> 0,038; price@1k[€] (none) -> 0,022
- C40, C5: Mfr.No: T520A107M006ATE045 -> T55A107M6R3C0045; price@100[€] (none) -> 0,418; price@10[€] (none) -> 0,739; price@1k[€] (none) -> 0,369
- C47: Mfr.No: (none) -> C0603X5R1E104K030BB; Spannung 6,3V -> 25V; price@100[€] (none) -> 0,037; price@10[€] (none) -> 0,03; price@1k[€] (none) -> 0,022
- C48: price@100[€] (none) -> 0,718; price@10[€] (none) -> 0,432; price@1k[€] (none) -> 0,381
- C49: Mfr.No: T58MM226M6R3C0300 -> TCSOM0J476M8R-ZM1; price@100[€] (none) -> 0,781; price@10[€] (none) -> 0,432; price@1k[€] (none) -> 0,381
- C50, C51, C52, C53: Mfr.No: (none) -> C0402C225M9PACTU; price@100[€] (none) -> 0,093; price@10[€] (none) -> 0,08; price@1k[€] (none) -> 0,043
- C6: Mfr.No: (none) -> AMK107ABJ106KAHT; Spannung 25V -> 6,3V; price@100[€] (none) -> 0,053; price@10[€] (none) -> 0,149; price@1k[€] (none) -> 0,041
- D1: Mfr.No: (none) -> SML-LX0201UPGC-TR; price@100[€] (none) -> 0,224; price@10[€] (none) -> 0,091; price@1k[€] (none) -> 0,075
- D2: value D_Schottky -> SBR1A30T5-7; footprint Diode_SMD:D_0402_1005Metric -> Diode_SMD:D_SOD-523; Mfr.No: (none) -> SBR1A30T5-7; price@100[€] (none) -> 0,197; price@10[€] (none) -> 0,317; price@1k[€] (none) -> 0,125
- D3: Mfr.No: (none) -> SML-LX0201USBC-TR; price@100[€] (none) -> 0,218; price@10[€] (none) -> 0,088; price@1k[€] (none) -> 0,073
- D4: value Red -> White; Mfr.No: (none) -> SML-LX0201NWD-TR; price@100[€] (none) -> 0,273; price@10[€] (none) -> 0,121; price@1k[€] (none) -> 0,096
- FB1, FB2, FB3, FB4, FB5, FB6: value 220R@100Mhz -> 120R@100Mhz; Mfr.No: BLM18SG221TN1D -> BLM18SG121TN1D; price@100[€] (none) -> 0,064; price@10[€] (none) -> 0,043; price@1k[€] (none) -> 0,039
- J1: price@100[€] (none) -> 0,667; price@10[€] (none) -> 0,618; price@1k[€] (none) -> 0,488
- J2, J3, J4, J5, J6: price@100[€] (none) -> 0,36; price@10[€] (none) -> 0,315; price@1k[€] (none) -> 0,247
- L1: price@100[€] (none) -> 0,333; price@10[€] (none) -> 0,237; price@1k[€] (none) -> 0,171
- L2: price@100[€] (none) -> 0,281; price@10[€] (none) -> 0,211; price@1k[€] (none) -> 0,145
- L3: Mfr.No: LPWI252010B1R0T -> SRP2512A-1R0M; price@100[€] (none) -> 0,333; price@10[€] (none) -> 0,237; price@1k[€] (none) -> 0,171
- L4: Mfr.No: (none) -> MLG0603P39NHT000; price@100[€] (none) -> 0,032; price@10[€] (none) -> 0,029; price@1k[€] (none) -> 0,021
- R1, R10, R11, R2, R21, R22, R48, R5, R58, R9: footprint Resistor_SMD:R_0201_0603Metric -> ultimateFC:R_0201_0603Metric_mod; price@100[€] (none) -> 0,05; price@10[€] (none) -> 0,02; price@1k[€] (none) -> 0,01
- R3, R6: price@100[€] (none) -> 0,05; price@10[€] (none) -> 0,02; price@1k[€] (none) -> 0,01
- R4: value R -> 10k; footprint Resistor_SMD:R_0201_0603Metric -> ultimateFC:R_0201_0603Metric_mod; price@100[€] (none) -> 0,05; price@10[€] (none) -> 0,02; price@1k[€] (none) -> 0,01
- R47: value 21k -> 10k; price@100[€] (none) -> 0,05; price@10[€] (none) -> 0,02; price@1k[€] (none) -> 0,01
- R49: Mfr.No: (none) -> CST0612-FC-R0005-E; price@100[€] (none) -> 0,466; price@10[€] (none) -> 0,336; price@1k[€] (none) -> 0,279
- R7: value R -> 470R; footprint Resistor_SMD:R_0201_0603Metric -> ultimateFC:R_0201_0603Metric_mod; price@100[€] (none) -> 0,05; price@10[€] (none) -> 0,02; price@1k[€] (none) -> 0,01
- R8: value R -> 1k; footprint Resistor_SMD:R_0201_0603Metric -> ultimateFC:R_0201_0603Metric_mod; price@100[€] (none) -> 0,05; price@10[€] (none) -> 0,02; price@1k[€] (none) -> 0,01
- RN1, RN16, RN2, RN7: value 10k -> 15k; Mfr.No: (none) -> TC124-FR-0715KL; price@100[€] (none) -> 0,167; price@10[€] (none) -> 0,056; price@1k[€] (none) -> 0,028
- RN13, RN14, RN15, RN18, RN20, RN5, RN6, RN9: value 2k -> 2k2; Mfr.No: (none) -> YC104-FR-072K2L; price@100[€] (none) -> 0,161; price@10[€] (none) -> 0,053; price@1k[€] (none) -> 0,027
- TP29: value pad -> bridge; footprint TestPoint:TestPoint_Pad_1.0x1.0mm -> ultimateFC:solderbridge_tiny; symbol Connector:TestPoint_Alt -> Device:Jumper
- U1, U2, U24, U6: Mfr.No: (none) -> EFM8BB21F16G-C-QFN20R; price@100[€] (none) -> 0,59; price@10[€] (none) -> 0,556; price@1k[€] (none) -> 0,556
- U10, U12, U16, U17, U18, U19, U25, U27, U28, U3, U7, U9: Mfr.No: (none) -> NCP81253MNTBG; price@100[€] (none) -> 0,64; price@10[€] (none) -> 0,413; price@1k[€] (none) -> 0,272
- U11, U13, U15, U20, U21, U22, U23, U26, U29, U30, U4, U8: Mfr.No: (none) -> SIZ200DT-T1-GE3; price@100[€] (none) -> 0,526; price@10[€] (none) -> 0,365; price@1k[€] (none) -> 0,328
- U14: price@100[€] (none) -> 1,01; price@10[€] (none) -> 0,734; price@1k[€] (none) -> 0,478
- U31: Mfr.No: (none) -> INA186A2IDCKR; price@100[€] (none) -> 1,12; price@10[€] (none) -> 0,811; price@1k[€] (none) -> 0,529
- U32: price@100[€] (none) -> 8,88; price@10[€] (none) -> 7,50; price@1k[€] (none) -> 7,13
- U33: price@100[€] (none) -> 8,88; price@10[€] (none) -> 7,5; price@1k[€] (none) -> 7,13
- U34: price@100[€] (none) -> 2,387; price@10[€] (none) -> 2,255; price@1k[€] (none) -> 2,18
- U35: price@100[€] (none) -> 29; price@10[€] (none) -> 14,7; price@1k[€] (none) -> 14,7
- U36: price@100[€] (none) -> 2,26; price@10[€] (none) -> 1,59; price@1k[€] (none) -> 1,25
- U37: price@100[€] (none) -> 2,25; price@10[€] (none) -> 1,97; price@1k[€] (none) -> 1,75
- U39: price@100[€] (none) -> 2,30; price@10[€] (none) -> 1,61; price@1k[€] (none) -> 1,26
- U5: price@100[€] (none) -> 2,1; price@10[€] (none) -> 1,58; price@1k[€] (none) -> 1,07
- X1: price@100[€] (none) -> 0,445; price@10[€] (none) -> 0,39; price@1k[€] (none) -> 0,306
- Y1: price@100[€] (none) -> 0,184; price@10[€] (none) -> 0,147; price@1k[€] (none) -> 0,131
- Y2: value 27M -> ECS-270-8-47Q-CES-TR; footprint Crystal:Crystal_SMD_MicroCrystal_CM9V-T1A-2Pin_1.6x1.0mm -> ultimateFC:ECX-1247Q; symbol Device:Crystal_Small -> Device:Crystal_GND24; Mfr.No: (none) -> ECS-270-8-47Q-CES-TR; price@100[€] (none) -> 0,548; price@10[€] (none) -> 0,452; price@1k[€] (none) -> 0,375
Connections:
- net labels added: USB_VBUS
- wire segments 862 -> 889
Other:
- note added: "3300mV (ref) / (1k/(1k+10k))\n=36,3 Fullscale"
- note added: "3300mV (ref) / 50 =66mV\n66mV/0.5mR =132A Fullscale"
- note added: "Added switch-off Transistor\nwhen supplied with USB\nJumper for continous supply"
- note added: "Is connetec to fiducial"
- note added: "TFM252012ALMA1R0MTAA as alternative"
- note added: "The Diode ond the resistors have to be selected\nthat USB_VBUS doesnt charge up over 2 V \neven at very high Temp"
- note removed: "1200mV (ref) / (1k/(1k+21k))\n=26,4V Fullscale"
- note removed: "1200mV (ref) / 25 =48mV\n48mV/0.5mR =96A Fullscale"
- note removed: "Add 2k7 pulldown"
- note removed: "Specify Quartz"
- note removed: "Wechsel auf TFM252012ALMA1R0MTAA wär nicht verkehrt"
- note removed: "connect to castellated pad"
- note removed: "issue #1"
- note removed: "issue #2"
- note removed: "only very small headroom of INA185A2 for 6S (26V max)\nChange to INA186-Q1 in SC70 package!\n\n"
- moved on the sheet: C12, C13, C14, C15, C20, C21, C24, C25, C26, C27, C41, C42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
